Commit message: Imported Actual Exomy Model
Co-authored-by: abmoRobotics <abmoRobotics@users.noreply.github.com>
Co-authored-by: mariebogestrand <mariebogestrand@users.noreply.github.com>
Co-authored-by: etpe19 <etpe19@users.noreply.github.com>

File: assets/urdf/exomy_modelv2/urdf/exomy_model.urdf (robot description, URDF)
Before this commit: robot Exomy_URDF, 19 links, 18 joints
Links:
- link 3D_Cam: mass 0.10791 -> 0.075
- link CL_Drive: mass 0.059839 -> 0.06
- link CL_Steer: mass 0.0714737501116116 -> 0.0735
- link CR_Drive: mass 0.059839 -> 0.060
- link CR_Steer: mass 0.0721879173626643 -> 0.0735
- link FL_Drive: mass 0.059839 -> 0.06
- link FL_Steer: mass 0.0721879173626638 -> 0.0735
- link FR_Drive: mass 0.059839 -> 0.06
- link FR_Steer: mass 0.0714737501116121 -> 0.0735
- link Left_Bogie: mass 0.0945481157691983 -> 0.1165
- link Mast: mass 0.0635336585695427 -> 0.057
- link RL_Drive: mass 0.059839 -> 0.06
- link RL_Steer: mass 0.072188 -> 0.0735
- link RR_Drive: mass 0.059839 -> 0.06
- link RR_Steer: mass 0.0714737501116104 -> 0.0735
- link Rear_Bogie: mass 0 -> 0.1165
- link Right_Bogie: mass 0.094548 -> 0.1165
- link Tracking_Cam: mass 0.015352 -> 0.060
Joints:
- joint Right_Bogie_Joint: axis -1 0 0 -> 0 0 1

Commit message: dof_force_tensor

File: assets/urdf/exomy_modelv2/urdf/exomy_model.urdf (robot description, URDF)
Before this commit: robot Exomy_URDF, 19 links, 18 joints
Joints:
- joint Left_Bogie_Joint: limit lower=-0.47 upper=0.47 velocity=1.0 -> lower=-0.47 upper=0.47 effort=0.0 velocity=1.0
- joint Rear_Bogie_Joint: limit lower=-0.47 upper=0.47 velocity=1.0 -> lower=-0.47 upper=0.47 effort=0.0 velocity=1.0
- joint Right_Bogie_Joint: limit lower=-0.47 upper=0.47 velocity=1.0 -> lower=-0.47 upper=0.47 effort=0.0 velocity=1.0

Commit message: Check spawn slope, URDF mass adjusted

File: assets/urdf/exomy_modelv2/urdf/exomy_model.urdf (robot description, URDF)
Before this commit: robot Exomy_URDF, 19 links, 18 joints
Links:
- link 3D_Cam: mass 0.075 -> 0.005
- link Mast: mass 0.057 -> 0.005
- link Tracking_Cam: mass 0.060 -> 0.005
